Commit message: fix gripper

File: urdf/Piper_2_Dummy2.xacro (robot description, xacro)
@@ -171,5 +171,5 @@
   </inertial>
   <visual>
-    <origin xyz="0.005706 -0.787489 0.001118" rpy="0 0 0"/>
+    <origin xyz="${0.005706-0.21798} ${-0.787489+0.394741} ${0.001118+0.40252}" rpy="0 0 0"/>
     <geometry>
       <mesh filename="file://$(find Piper_2_Dummy2_description)/meshes/piper_right_1.stl" scale="0.001 0.001 0.001"/>
@@ -178,5 +178,5 @@
   </visual>
   <collision>
-    <origin xyz="0.005706 -0.787489 0.001118" rpy="0 0 0"/>
+    <origin xyz="${0.005706-0.21798} ${-0.787489+0.394741} ${0.001118+0.40252}" rpy="0 0 0"/>
     <geometry>
       <mesh filename="file://$(find Piper_2_Dummy2_description)/meshes/piper_right_1.stl" scale="0.001 0.001 0.001"/>
@@ -191,5 +191,5 @@
   </inertial>
   <visual>
-    <origin xyz="0.005706 -0.787489 0.001118" rpy="0 0 0"/>
+    <origin xyz="${0.005706-0.21798} ${-0.787489+0.394741} ${0.001118+0.40252}" rpy="0 0 0"/>
     <geometry>
       <mesh filename="file://$(find Piper_2_Dummy2_description)/meshes/piper_left_1.stl" scale="0.001 0.001 0.001"/>
@@ -198,5 +198,5 @@
   </visual>
   <collision>
-    <origin xyz="0.005706 -0.787489 0.001118" rpy="0 0 0"/>
+    <origin xyz="${0.005706-0.21798} ${-0.787489+0.394741} ${0.001118+0.40252}" rpy="0 0 0"/>
     <geometry>
       <mesh filename="file://$(find Piper_2_Dummy2_description)/meshes/piper_left_1.stl" scale="0.001 0.001 0.001"/>
@@ -351,5 +351,5 @@
   </inertial>
   <visual>
-    <origin xyz="0.005754 -0.794109 0.001137" rpy="0 0 0"/>
+    <origin xyz="${0.005754+0.202975} ${-0.794109+0.401161} ${0.001137+0.402501}" rpy="0 0 0"/>
     <geometry>
       <mesh filename="file://$(find Piper_2_Dummy2_description)/meshes/piper_right_L_1.stl" scale="0.001 0.001 0.001"/>
@@ -358,5 +358,5 @@
   </visual>
   <collision>
-    <origin xyz="0.005754 -0.794109 0.001137" rpy="0 0 0"/>
+    <origin xyz="${0.005754+0.202975} ${-0.794109+0.401161} ${0.001137+0.402501}" rpy="0 0 0"/>
     <geometry>
       <mesh filename="file://$(find Piper_2_Dummy2_description)/meshes/piper_right_L_1.stl" scale="0.001 0.001 0.001"/>
@@ -371,5 +371,5 @@
   </inertial>
   <visual>
-    <origin xyz="0.005754 -0.794109 0.001137" rpy="0 0 0"/>
+    <origin xyz="${0.005754+0.202975} ${-0.794109+0.401161} ${0.001137+0.402501}" rpy="0 0 0"/>
     <geometry>
       <mesh filename="file://$(find Piper_2_Dummy2_description)/meshes/piper_left_L_1.stl" scale="0.001 0.001 0.001"/>
@@ -378,5 +378,5 @@
   </visual>
   <collision>
-    <origin xyz="0.005754 -0.794109 0.001137" rpy="0 0 0"/>
+    <origin xyz="${0.005754+0.202975} ${-0.794109+0.401161} ${0.001137+0.402501}" rpy="0 0 0"/>
     <geometry>
       <mesh filename="file://$(find Piper_2_Dummy2_description)/meshes/piper_left_L_1.stl" scale="0.001 0.001 0.001"/>
@@ -652,5 +652,5 @@
 </joint>
 <joint name="Slider _9_R" type="prismatic">
-  <origin xyz="-0.21798 0.394741 0.40252" rpy="0 0 0"/>
+  <origin xyz="${0} ${0} ${0}" rpy="0 0 0"/>
   <parent link="piper_hand_1"/>
   <child link="piper_right_1"/>
@@ -659,5 +659,5 @@
 </joint>
 <joint name="Slider_10_R" type="prismatic">
-  <origin xyz="-0.21798 0.394741 0.40252" rpy="0 0 0"/>
+  <origin xyz="${0} ${0} ${0}" rpy="0 0 0"/>
   <parent link="piper_hand_1"/>
   <child link="piper_left_1"/>
@@ -713,5 +713,5 @@
 </joint>
 <joint name="Slider_9_L" type="prismatic">
-  <origin xyz="0.202975 0.401161 0.402501" rpy="0 0 0"/>
+  <origin xyz="${0} ${0} ${0}" rpy="0 0 0"/>
   <parent link="piper_hand_L_1"/>
   <child link="piper_right_L_1"/>
@@ -720,5 +720,5 @@
 </joint>
 <joint name="Slider_10_L" type="prismatic">
-  <origin xyz="0.202975 0.401161 0.402501" rpy="0 0 0"/>
+  <origin xyz="${0} ${0} ${0}" rpy="0 0 0"/>
   <parent link="piper_hand_L_1"/>
   <child link="piper_left_L_1"/>

Commit message: name change

File: urdf/Piper_2_Dummy2.xacro (robot description, xacro)
@@ -424,5 +424,5 @@
   </collision>
 </link>
-<link name="墊片_v3_1">
+<link name="shim">
   <inertial>
     <origin xyz="-2.603155605204514e-13 0.04987462633751475 0.022990960314565406" rpy="0 0 0"/>
@@ -433,5 +433,5 @@
     <origin xyz="0.0 0.05 -0.0708" rpy="0 0 0"/>
     <geometry>
-      <mesh filename="file://$(find Piper_2_Dummy2_description)/meshes/墊片_v3_1.stl" scale="0.001 0.001 0.001"/>
+      <mesh filename="file://$(find Piper_2_Dummy2_description)/meshes/shim.stl" scale="0.001 0.001 0.001"/>
     </geometry>
     <material name="silver"/>
@@ -440,5 +440,5 @@
     <origin xyz="0.0 0.05 -0.0708" rpy="0 0 0"/>
     <geometry>
-      <mesh filename="file://$(find Piper_2_Dummy2_description)/meshes/墊片_v3_1.stl" scale="0.001 0.001 0.001"/>
+      <mesh filename="file://$(find Piper_2_Dummy2_description)/meshes/shim.stl" scale="0.001 0.001 0.001"/>
     </geometry>
   </collision>
@@ -564,5 +564,5 @@
   </collision>
 </link>
-<link name="435_支架_v2_1">
+<link name="bracket_435">
   <inertial>
     <origin xyz="-7.328758401016489e-08 0.00408106128329172 -1.0980955755801602e-08" rpy="0 0 0"/>
@@ -573,5 +573,5 @@
     <origin xyz="-0.013149 -0.26281 -0.452482" rpy="0 0 0"/>
     <geometry>
-      <mesh filename="file://$(find Piper_2_Dummy2_description)/meshes/435_支架_v2_1.stl" scale="0.001 0.001 0.001"/>
+      <mesh filename="file://$(find Piper_2_Dummy2_description)/meshes/bracket_435.stl" scale="0.001 0.001 0.001"/>
     </geometry>
     <material name="silver"/>
@@ -580,5 +580,5 @@
     <origin xyz="-0.013149 -0.26281 -0.452482" rpy="0 0 0"/>
     <geometry>
-      <mesh filename="file://$(find Piper_2_Dummy2_description)/meshes/435_支架_v2_1.stl" scale="0.001 0.001 0.001"/>
+      <mesh filename="file://$(find Piper_2_Dummy2_description)/meshes/bracket_435.stl" scale="0.001 0.001 0.001"/>
     </geometry>
   </collision>
@@ -651,5 +651,5 @@
   <child link="piper_hand_1"/>
 </joint>
-<joint name="Slider _9_R" type="prismatic">
+<joint name="Slider_9_R" type="prismatic">
   <origin xyz="${0} ${0} ${0}" rpy="0 0 0"/>
   <parent link="piper_hand_1"/>
@@ -736,12 +736,12 @@
   <child link="piper_R_base_1"/>
 </joint>
-<joint name="Rigid 77" type="fixed">
+<joint name="Rigid_77" type="fixed">
   <origin xyz="0.0 -0.05 0.0708" rpy="0 0 0"/>
   <parent link="base_link"/>
-  <child link="墊片_v3_1"/>
+  <child link="shim"/>
 </joint>
 <joint name="Rigid 78" type="fixed">
   <origin xyz="0.0 0.0 0.026" rpy="0 0 0"/>
-  <parent link="墊片_v3_1"/>
+  <parent link="shim"/>
   <child link="dummy2_link0_v1_1"/>
 </joint>
@@ -784,5 +784,5 @@
   <origin xyz="-0.021 0.1185 0.0" rpy="0 0 0"/>
   <parent link="link6_v1_1"/>
-  <child link="435_支架_v2_1"/>
+  <child link="bracket_435"/>
   <axis xyz="0.0 -1.0 -0.0"/>
   <limit upper="3.141593" lower="-3.141593" effort="100" velocity="100"/>
@@ -790,5 +790,5 @@
 <joint name="Rigid 85" type="fixed">
   <origin xyz="0.0225 0.007 0.0" rpy="0 0 0"/>
-  <parent link="435_支架_v2_1"/>
+  <parent link="bracket_435"/>
   <child link="RealSense_D435_v1_1"/>
 </joint>
